Commit message: Rework URDF and update movement

File: src/atom/urdf/atom.urdf (robot description, URDF)
Before this commit: robot atom, 9 links, 8 joints
Links:
- removed link left_wheel_front
- removed link right_wheel_front
- added link left_wheel, mass 5; collision cylinder length=0.1 radius=0.157226; visual cylinder length=0.1 radius=0.157226
- added link right_wheel, mass 5; collision cylinder length=0.1 radius=0.157226; visual cylinder length=0.1 radius=0.157226
Joints:
- removed joint left_wheel_hinge_front
- removed joint right_wheel_hinge_front
- added joint left_wheel_joint: type continuous, parent chassis, child left_wheel, origin xyz=0.3 0.36 -0.2794 rpy=0 0 0, axis 0 1 0
- added joint right_wheel_joint: type continuous, parent chassis, child right_wheel, origin xyz=0.3 -0.36 -0.2794 rpy=0 0 0, axis 0 1 0
- joint robot_footprint_joint: origin xyz=0 0 0.436626 rpy=0 0 0 -> xyz=0 0 0.43682599999999994 rpy=0 0 0

File: src/atom/urdf/atom.xacro (robot description, xacro)
@@ -1,15 +1,28 @@
 <?xml version='1.0'?>
+<!-- TODO: Switch back to 4 wheel skid steer drive -->
 <robot name="atom" xmlns:xacro="http://www.ros.org/wiki/xacro">
-	<xacro:property name="robot_name" value="atom" />
-	<xacro:property name="robot_chassis_mass" value="29.9371" />
-	<xacro:property name="robot_wheel_mass" value="5" />
-	<xacro:property name="robot_wheel_length" value="0.1" />
-	<xacro:property name="robot_wheel_radius" value="0.157226" />
+	<xacro:property name="height_offset" value="0.0002" /> <!-- How far the robot starts off the ground -->
+	<xacro:property name="front_offset" value="0.3" /> <!-- How far forward the wheels and lidar are compared to the center of the chassis -->
+	<xacro:property name="back_offset" value="-0.5715" /> <!-- How far back the caster wheel is compared to the center of the chassis -->
+	<xacro:property name="chassis_mass" value="29.9371" />
+	<xacro:property name="chassis_length" value="1.143" />
+	<xacro:property name="chassis_width" value="0.6096" />
+	<xacro:property name="chassis_height" value="0.5588" />
+	<xacro:property name="caster_radius" value="0.05" />
+	<xacro:property name="wheel_mass" value="5" />
+	<xacro:property name="wheel_radius" value="0.157226" />
+	<xacro:property name="wheel_width" value="0.1" />
+	<xacro:property name="wheel_separation" value="0.72" /> <!-- Distance from center to center -->
 	<xacro:property name="camera_mass" value="0.1"/>
-	<!-- Make Chassis of Bot -->
+	<xacro:property name="camera_front_offset" value="0.5715"/> <!-- How far forward the camera is compared to the center of the chassis -->
+	<xacro:property name="camera_z_offset" value="-0.2"/> <!-- How far down the camera is compared to the center of the chassis -->
+	<xacro:property name="lidar_height" value="0.89535"/> <!-- The distance from the base of the chassis to the base of the LiDAR -->
+	<!-- Robot footprint on ground -->
+	<link name="robot_footprint" />
+	<!-- Chassis -->
 	<link name="chassis">
 		<pose>0.536448 -0.130302 0.066802 0 0 0</pose>
 		<inertial>
-			<mass value="${robot_chassis_mass}" />
+			<mass value="${chassis_mass}" />
 			<origin xyz="0 0 0" rpy="0 0 0" />
 			<inertia
@@ -22,5 +35,5 @@
 			<origin xyz="0 0 0" rpy="0 0 0" />
 			<geometry>
-				<box size="1.143 0.6096 0.5588" />
+				<box size="${chassis_length} ${chassis_width} ${chassis_height}" />
 			</geometry>
 		</collision>
@@ -28,11 +41,11 @@
 			<origin xyz="0 0 0" rpy="0 0 0" />
 			<geometry>
-				<box size="1.143 0.6096 0.5588" />
+				<box size="${chassis_length} ${chassis_width} ${chassis_height}" />
 			</geometry>
 		</visual>
 		<collision name='caster_collision'>
-			<origin xyz="-0.5715 0 -0.386626" rpy=" 0 0 0"/>
+			<origin xyz="${back_offset} 0 ${-chassis_height/2-wheel_radius+caster_radius}" rpy=" 0 0 0"/>
 			<geometry>
-				<sphere radius="0.05"/>
+				<sphere radius="${caster_radius}"/>
 			</geometry>
 			<surface>
@@ -48,117 +61,30 @@
 		</collision>
 		<visual name='caster_visual'>
-			<origin xyz="-0.5715 0 -0.386626" rpy=" 0 0 0"/>
+			<origin xyz="${back_offset} 0 ${-chassis_height/2-wheel_radius+caster_radius}" rpy=" 0 0 0"/>
 			<geometry>
-				<sphere radius="0.05"/>
+				<sphere radius="${caster_radius}"/>
 			</geometry>
 		</visual>
 	</link>
-	<!-- Right Wheel Front-->
-	<link name="right_wheel_front">
-		<inertial>
-			<mass value="${robot_wheel_mass}" />
-			<origin xyz="0 0 0" rpy="0 1.5707 1.5707" />
-			<inertia
-				ixx="0.03506668551166666666666666666667" ixy="0.0" ixz="0.0"
-				iyy="0.03506668551166666666666666666667" iyz="0.0"
-				izz="0.030900018845"
-			/>
-		</inertial>
-		<visual>
-			<origin xyz="0 0 0" rpy="0 1.5707 1.5707" />
-			<geometry>
-				<cylinder radius="${robot_wheel_radius}" length="${robot_wheel_length}" />
-			</geometry>
-		</visual>
-		<collision>
-			<origin xyz="0 0 0" rpy="0 1.5707 1.5707" />
-			<geometry>
-				<cylinder radius="${robot_wheel_radius}" length="${robot_wheel_length}" />
-			</geometry>
-		</collision>
-	</link>
-	<!-- Left wheel Front-->
-	<link name="left_wheel_front">
-		<inertial>
-			<mass value="${robot_wheel_mass}" />
-			<origin xyz="0 0 0" rpy="0 1.5707 1.5707" />
-			<inertia
-				ixx="0.03506668551166666666666666666667" ixy="0.0" ixz="0.0"
-				iyy="0.03506668551166666666666666666667" iyz="0.0"
-				izz="0.030900018845"
-			/>
-		</inertial>
-		<visual>
-			<origin xyz="0 0 0" rpy="0 1.5707 1.5707" />
-			<geometry>
-				<cylinder radius="${robot_wheel_radius}" length="${robot_wheel_length}" />
-			</geometry>
-		</visual>
-		<collision>
-			<origin xyz="0 0 0" rpy="0 1.5707 1.5707" />
-			<geometry>
-				<cylinder radius="${robot_wheel_radius}" length="${robot_wheel_length}" />
-			</geometry>
-		</collision>
-	</link>
+	<!-- Wheels -->
+	<xacro:include filename="$(find atom)/urdf/wheel.xacro"/>
+	<xacro:wheel prefix="right" mass="${wheel_mass}" radius="${wheel_radius}" width="${wheel_width}">
+		<origin xyz="${front_offset} -${wheel_separation/2} ${-chassis_height/2}" rpy="0 0 0" />
+	</xacro:wheel>
+	<xacro:wheel prefix="left" mass="${wheel_mass}" radius="${wheel_radius}" width="${wheel_width}">
+		<origin xyz="${front_offset} ${wheel_separation/2} ${-chassis_height/2}" rpy="0 0 0" />
+	</xacro:wheel>
 	<!-- Camera -->
-	<link name="camera">
-		<inertial>
-			<mass value="${camera_mass}"/>
-			<origin xyz="0 0 0" rpy="0 0 0"/>
-			<inertia
-		        ixx="1e-6" ixy="0.0" ixz="0.0"
-		        iyy="1e-6" iyz="0.0"
-		        izz="1e-6"
-		      />
-		</inertial>
-		<visual>
-			<origin xyz="0 0 0" rpy="0 0 0"/>
-			<geometry>
-				<box size="0.05 0.05 0.05"/>
-			</geometry>
-		</visual>
-		<collision>
-			<origin xyz="0 0 0" rpy="0 0 0"/>
-			<geometry>
-				<box size="0.05 0.05 0.05"/>
-			</geometry>
-		</collision>
-	</link>
-	<link name="camera_link_optical" />
+	<xacro:include filename="$(find atom)/urdf/camera.xacro"/>
+	<xacro:camera mass="${camera_mass}">
+		<origin xyz="${camera_front_offset} 0 ${camera_z_offset}" rpy="0 0 0" />
+	</xacro:camera>
+	<!-- LiDAR -->
+	<xacro:include filename="$(find velodyne_description)/urdf/VLP-16.urdf.xacro" />
+	<xacro:VLP-16 parent="chassis" name="velodyne" topic="/points2" hz="10" samples="250" gpu="false">
+		<origin xyz="${front_offset} 0 ${-chassis_height/2+lidar_height}" rpy="0 0 0" />
+	</xacro:VLP-16>
+	<!-- IMU -->
 	<link name="imu_link" />
-	<!-- Project center to the ground -->
-	<link name="robot_footprint" />
-	<!-- Define Joints -->
-	<!-- Right Wheel Joint Front-->
-	<joint type="continuous" name="right_wheel_hinge_front">
-		<origin xyz="0.3 -0.3548 -0.2794" rpy="0 0 0" />
-		<parent link="chassis" />
-		<child link="right_wheel_front" />
-		<axis xyz="0 1 0" rpy="0 0 0" />
-		<limit effort="10000" velocity="1000" />
-		<dynamics damping="1.0" friction="1.0" />
-	</joint>
-	<!-- Left Wheel Joint Front-->
-	<joint type="continuous" name="left_wheel_hinge_front">
-		<origin xyz="0.3 0.3548 -0.2794" rpy="0 0 0" />
-		<parent link="chassis" />
-		<child link="left_wheel_front" />
-		<axis xyz="0 1 0" rpy="0 0 0" />
-		<limit effort="10000" velocity="1000" />
-		<dynamics damping="1.0" friction="1.0" />
-	</joint>
-	<!-- Camera Joint -->
-	<joint name="camera_joint" type="fixed">
-		<origin xyz="0.5715 0 -0.2" rpy="0 0 0" />
-		<parent link="chassis" />
-		<child link="camera" />
-		<axis xyz="0 1 0" />
-	</joint>
-	<joint name="camera_optical_joint" type="fixed">
-		<origin xyz="0 0 0" rpy="${-pi/2} 0 ${-pi/2}"/>
-		<parent link="camera" />
-		<child link="camera_link_optical" />
-	</joint>
 	<!-- IMU Joint -->
 	<joint name="imu_joint" type="fixed">
@@ -168,53 +94,15 @@
 		<axis xyz="0 1 0" />
 	</joint>
+	<!-- Chassis Joint -->
 	<joint name="robot_footprint_joint" type="fixed">
-		<origin xyz="0 0 0.436626" rpy="0 0 0" />
+		<origin xyz="0 0 ${chassis_height/2+wheel_radius+height_offset}" rpy="0 0 0" />
 		<parent link="robot_footprint" />
 		<child link="chassis" />
 	</joint>
 	<!-- Color of bot -->
-	<gazebo reference="left_wheel_front">
-		<material>Gazebo/Green</material>
-		<kp>1000000.0</kp> <!-- kp and kd for rubber -->
-		<kd>100.0</kd>
-		<mu1>1.0</mu1>
-		<mu2>1.0</mu2>
-		<maxVel>1.0</maxVel>
-		<minDepth>0.00</minDepth>
-	</gazebo>
-	<gazebo reference="middle_wheel_back">
-		<material>Gazebo/Green</material>
-		<kp>1000000.0</kp> <!-- kp and kd for rubber -->
-		<kd>100.0</kd>
-		<mu1>1.0</mu1>
-		<mu2>1.0</mu2>
-		<maxVel>1.0</maxVel>
-		<minDepth>0.00</minDepth>
-	</gazebo>
-	<gazebo reference="right_wheel_front">
-		<material>Gazebo/Green</material>
-		<kp>1000000.0</kp> <!-- kp and kd for rubber -->
-		<kd>100.0</kd>
-		<mu1>1.0</mu1>
-		<mu2>1.0</mu2>
-		<maxVel>1.0</maxVel>
-		<minDepth>0.00</minDepth>
-	</gazebo>
-	<gazebo reference="camera">
-		<material>Gazebo/Red</material>
-	</gazebo>
 	<gazebo reference="chassis">
 		<material>Gazebo/Blue</material>
 	</gazebo>
-	<!-- including the LiDAR xacro file and creating an instance of it -->
-	<!-- somehow the xacro needs to be in the VLP-16 tags for it to show up -->
-	<xacro:include
-		filename="$(find velodyne_description)/urdf/VLP-16.urdf.xacro" />
-	<xacro:VLP-16 parent="chassis" name="velodyne" topic="/points2" hz="10" samples="250"
-		gpu="false">
-		<origin xyz="0.3 0 0.61595" rpy="0 0 0" /> <!-- samples 440-->
-		<!-- the height number needs to be adjusted -->
-	</xacro:VLP-16>
-	<!-- Motor, Camera and Lidar Simulation -->
+	<!-- Motor, Camera and IMU Simulation -->
 	<xacro:include filename="$(find atom)/urdf/atom.gazebo" />
 </robot>

Commit message: Improve movement and update urdf

File: src/atom/urdf/atom.urdf (robot description, URDF)
Before this commit: robot atom, 9 links, 8 joints
Links:
- removed link robot_footprint
- added link base_footprint
- added link chassis_inertial_link, mass 29.9371
- link chassis: mass 29.9371 -> None
- link left_wheel: geometry collision cylinder length=0.15 radius=0.157226; visual cylinder length=0.15 radius=0.157226
- link right_wheel: geometry collision cylinder length=0.15 radius=0.157226; visual cylinder length=0.15 radius=0.157226
Joints:
- removed joint robot_footprint_joint
- added joint base_footprint_joint: type fixed, parent chassis, child base_footprint, origin xyz=0 0 -0.42662599999999995 rpy=0 0 0
- added joint chassis_inertial_joint: type fixed, parent chassis, child chassis_inertial_link, origin xyz=0 0 0 rpy=0 0 0
- joint left_wheel_joint: limit (none) -> effort=1000 velocity=1000; origin xyz=0.3 0.36 -0.2794 rpy=0 0 0 -> xyz=0.3 0.39 -0.2694 rpy=0 0 0
- joint right_wheel_joint: limit (none) -> effort=1000 velocity=1000; origin xyz=0.3 -0.36 -0.2794 rpy=0 0 0 -> xyz=0.3 -0.39 -0.2694 rpy=0 0 0

File: src/atom/urdf/atom.xacro (robot description, xacro)
@@ -1,6 +1,4 @@
 <?xml version='1.0'?>
-<!-- TODO: Switch back to 4 wheel skid steer drive -->
 <robot name="atom" xmlns:xacro="http://www.ros.org/wiki/xacro">
-	<xacro:property name="height_offset" value="0.0002" /> <!-- How far the robot starts off the ground -->
 	<xacro:property name="front_offset" value="0.3" /> <!-- How far forward the wheels and lidar are compared to the center of the chassis -->
 	<xacro:property name="back_offset" value="-0.5715" /> <!-- How far back the caster wheel is compared to the center of the chassis -->
@@ -9,9 +7,14 @@
 	<xacro:property name="chassis_width" value="0.6096" />
 	<xacro:property name="chassis_height" value="0.5588" />
+	<!-- Center of mass -->
+	<xacro:property name="com_x" value="0" />
+	<xacro:property name="com_y" value="0" />
+	<xacro:property name="com_z" value="0" />
 	<xacro:property name="caster_radius" value="0.05" />
 	<xacro:property name="wheel_mass" value="5" />
 	<xacro:property name="wheel_radius" value="0.157226" />
-	<xacro:property name="wheel_width" value="0.1" />
-	<xacro:property name="wheel_separation" value="0.72" /> <!-- Distance from center to center -->
+	<xacro:property name="wheel_width" value="0.15" />
+	<xacro:property name="wheel_separation" value="0.78" /> <!-- Distance from center to center -->
+	<xacro:property name="wheel_offset" value="0.01" /> <!-- How far above the bottom plate of the robot the wheels are -->
 	<xacro:property name="camera_mass" value="0.1"/>
 	<xacro:property name="camera_front_offset" value="0.5715"/> <!-- How far forward the camera is compared to the center of the chassis -->
@@ -19,17 +22,8 @@
 	<xacro:property name="lidar_height" value="0.89535"/> <!-- The distance from the base of the chassis to the base of the LiDAR -->
 	<!-- Robot footprint on ground -->
-	<link name="robot_footprint" />
+	<link name="base_footprint" />
 	<!-- Chassis -->
 	<link name="chassis">
-		<pose>0.536448 -0.130302 0.066802 0 0 0</pose>
-		<inertial>
-			<mass value="${chassis_mass}" />
-			<origin xyz="0 0 0" rpy="0 0 0" />
-			<inertia
-				ixx="1.699" ixy="0" ixz="0"
-				iyy="4.022" iyz="0"
-				izz="4.170"
-			/>
-		</inertial>
+		<origin xyz="0 0 0" rpy="0 0 0" />
 		<collision name="collision">
 			<origin xyz="0 0 0" rpy="0 0 0" />
@@ -45,5 +39,5 @@
 		</visual>
 		<collision name='caster_collision'>
-			<origin xyz="${back_offset} 0 ${-chassis_height/2-wheel_radius+caster_radius}" rpy=" 0 0 0"/>
+			<origin xyz="${back_offset} 0 ${caster_radius+wheel_offset-wheel_radius-chassis_height/2}" rpy=" 0 0 0"/>
 			<geometry>
 				<sphere radius="${caster_radius}"/>
@@ -52,8 +46,6 @@
 				<friction>
 				<ode>
-					<mu>1</mu>
-					<mu2>1</mu2>
-					<slip1>0.5</slip1>
-					<slip2>0</slip2>
+					<mu>0.0</mu>
+					<mu2>0.0</mu2>
 				</ode>
 				</friction>
@@ -61,5 +53,5 @@
 		</collision>
 		<visual name='caster_visual'>
-			<origin xyz="${back_offset} 0 ${-chassis_height/2-wheel_radius+caster_radius}" rpy=" 0 0 0"/>
+			<origin xyz="${back_offset} 0 ${caster_radius+wheel_offset-wheel_radius-chassis_height/2}" rpy=" 0 0 0"/>
 			<geometry>
 				<sphere radius="${caster_radius}"/>
@@ -67,11 +59,22 @@
 		</visual>
 	</link>
+	<link name="chassis_inertial_link">
+		<inertial>
+			<mass value="${chassis_mass}" />
+			<origin xyz="${com_x} ${com_y} ${com_z}" rpy="0 0 0" />
+			<inertia
+				ixx="${chassis_mass/12*(chassis_height**2+chassis_length**2)}" ixy="0" ixz="0"
+				iyy="${chassis_mass/12*(chassis_width**2+chassis_height**2)}" iyz="0"
+				izz="${chassis_mass/12*(chassis_width**2+chassis_length**2)}"
+			/>
+		</inertial>
+	</link>
 	<!-- Wheels -->
 	<xacro:include filename="$(find atom)/urdf/wheel.xacro"/>
 	<xacro:wheel prefix="right" mass="${wheel_mass}" radius="${wheel_radius}" width="${wheel_width}">
-		<origin xyz="${front_offset} -${wheel_separation/2} ${-chassis_height/2}" rpy="0 0 0" />
+		<origin xyz="${front_offset} -${wheel_separation/2} ${wheel_offset-chassis_height/2}" rpy="0 0 0" />
 	</xacro:wheel>
 	<xacro:wheel prefix="left" mass="${wheel_mass}" radius="${wheel_radius}" width="${wheel_width}">
-		<origin xyz="${front_offset} ${wheel_separation/2} ${-chassis_height/2}" rpy="0 0 0" />
+		<origin xyz="${front_offset} ${wheel_separation/2} ${wheel_offset-chassis_height/2}" rpy="0 0 0" />
 	</xacro:wheel>
 	<!-- Camera -->
@@ -82,6 +85,6 @@
 	<!-- LiDAR -->
 	<xacro:include filename="$(find velodyne_description)/urdf/VLP-16.urdf.xacro" />
-	<xacro:VLP-16 parent="chassis" name="velodyne" topic="/points2" hz="10" samples="250" gpu="false">
-		<origin xyz="${front_offset} 0 ${-chassis_height/2+lidar_height}" rpy="0 0 0" />
+	<xacro:VLP-16 parent="chassis" name="velodyne" topic="/points2" hz="20" samples="250" gpu="false">
+		<origin xyz="${front_offset} 0 ${lidar_height-chassis_height/2}" rpy="0 0 0" />
 	</xacro:VLP-16>
 	<!-- IMU -->
@@ -95,8 +98,14 @@
 	</joint>
 	<!-- Chassis Joint -->
-	<joint name="robot_footprint_joint" type="fixed">
-		<origin xyz="0 0 ${chassis_height/2+wheel_radius+height_offset}" rpy="0 0 0" />
-		<parent link="robot_footprint" />
-		<child link="chassis" />
+	<joint name="base_footprint_joint" type="fixed">
+		<origin xyz="0 0 ${wheel_offset-chassis_height/2-wheel_radius}" rpy="0 0 0" />
+		<parent link="chassis" />
+		<child link="base_footprint" />
+	</joint>
+	<!-- Chassis Inertial Joint -->
+	<joint name="chassis_inertial_joint" type="fixed">
+		<origin xyz="0 0 0" rpy="0 0 0" />
+		<parent link="chassis" />
+		<child link="chassis_inertial_link" />
 	</joint>
 	<!-- Color of bot -->

File: src/atom/urdf/wheel.xacro (robot description, xacro)
@@ -7,7 +7,7 @@
                 <origin xyz="0 0 0" rpy="0 ${pi/2} ${pi/2}" />
                 <inertia
-                    ixx="0.03506668551166666666666666666667" ixy="0.0" ixz="0.0"
-                    iyy="0.03506668551166666666666666666667" iyz="0.0"
-                    izz="0.030900018845"
+                    ixx="${mass/12*(3*radius**2+2*width**2)}" ixy="0.0" ixz="0.0"
+                    iyy="${mass/12*(3*radius**2+2*width**2)}" iyz="0.0"
+                    izz="${mass/2*radius**2}"
                 />
             </inertial>
@@ -30,12 +30,13 @@
             <child link="${prefix}_wheel" />
             <axis xyz="0 1 0" rpy="0 0 0" />
+            <limit effort="1000" velocity="1000"/>
+            <dynamics damping="0.0001"/>
         </joint>
         <gazebo reference="${prefix}_wheel">
             <material>Gazebo/Green</material>
             <mu1 value="1.0"/>
-            <mu2 value="0.5"/>
+            <mu2 value="1.0"/>
             <kp value="10000000.0" />
             <kd value="1.0" />
-            <fdir1 value="1 0 0"/>
             <maxVel>1.0</maxVel>
             <minDepth>0.00</minDepth>
